Commit message: Rvize,turn OK

File: rover_description/urdf/rover.gazebo.xacro (robot description, xacro)
@@ -9,24 +9,23 @@
   </gazebo>
   <gazebo>
-    <plugin name="differential_drive_controller" filename="libgazebo_ros_diff_drive.so">
-      <alwaysOn>true</alwaysOn>
-      <updateRate>100</updateRate>
-      <rosDebugLevel>Debug</rosDebugLevel>
-      <odometrySource>1</odometrySource>
-      <leftJoint>base_to_left1</leftJoint>
-      <rightJoint>base_to_right1</rightJoint>
+    <plugin name="skid_steer_drive_controller" filename="libgazebo_ros_skid_steer_drive.so">
+      <updateRate>100.0</updateRate>
+      <robotNamespace>/</robotNamespace>
+      <leftFrontJoint>base_to_left1</leftFrontJoint>
+      <rightFrontJoint>base_to_right1</rightFrontJoint>
       <leftRearJoint>base_to_left2</leftRearJoint>
       <rightRearJoint>base_to_right2</rightRearJoint>
-      <wheelSeparation>0.24</wheelSeparation>
-      <wheelDiameter>${wheel_diameter}</wheelDiameter>
-      <wheelTorque>0.8</wheelTorque>
-      <wheelAcceleration>0.05</wheelAcceleration>
+      <wheelSeparation>2</wheelSeparation>
+      <wheelDiameter>0.2</wheelDiameter>
+      <robotBaseFrame>base_link</robotBaseFrame>
+      <torque>20</torque>
+      <covariance_x>0.0001</covariance_x>
+      <covariance_y>0.0001</covariance_y>
+      <covariance_yaw>0.0001</covariance_yaw>
+      <topicName>cmd_vel</topicName>
+      <odometryFrame>odom</odometryFrame>
       <commandTopic>cmd_vel</commandTopic>
       <odometryTopic>odom</odometryTopic>
-      <odometryFrame>odom</odometryFrame>
-      <robotBaseFrame>base_footprint</robotBaseFrame>
-      <publishWheelTF>true</publishWheelTF>
-      <legacyMode>true</legacyMode>
-      <publishWheelJointState>true</publishWheelJointState>
+      <broadcastTF>true</broadcastTF>
     </plugin>
   </gazebo>

File: rover_description/urdf/rover.urdf.xacro (robot description, xacro)
@@ -33,4 +33,5 @@
   <link name="right_wheel1">
     <visual>
+      <origin xyz="0 0 0" rpy="0 0 ${PI}"/>
       <geometry>
         <mesh filename="file://${mesh_path}/meshes/14-010-p006.dae"/>
@@ -85,4 +86,5 @@
   <link name="right_wheel2">
     <visual>
+      <origin xyz="0 0 0" rpy="0 0 ${PI}"/>
       <geometry>
         <mesh filename="file://${mesh_path}/meshes/14-010-p006.dae"/>
@@ -138,5 +140,5 @@
     <type>transmission_interface/SimpleTransmission</type>
     <joint name="base_to_right1">
-      <hardwareInterface>EffortJointInterface</hardwareInterface>
+      <hardwareInterface>hardware_interface/EffortJointInterface</hardwareInterface>
     </joint>
     <actuator name="right_wheel1_motor">
@@ -146,5 +148,5 @@
     <type>transmission_interface/SimpleTransmission</type>
     <joint name="base_to_right2">
-      <hardwareInterface>EffortJointInterface</hardwareInterface>
+      <hardwareInterface>hardware_interface/EffortJointInterface</hardwareInterface>
     </joint>
     <actuator name="right_wheel2_motor">
@@ -154,5 +156,5 @@
     <type>transmission_interface/SimpleTransmission</type>
     <joint name="base_to_left1">
-      <hardwareInterface>EffortJointInterface</hardwareInterface>
+      <hardwareInterface>hardware_interface/EffortJointInterface</hardwareInterface>
     </joint>
     <actuator name="left_wheel1_motor">
@@ -162,5 +164,5 @@
     <type>transmission_interface/SimpleTransmission</type>
     <joint name="base_to_left2">
-      <hardwareInterface>EffortJointInterface</hardwareInterface>
+      <hardwareInterface>hardware_interface/EffortJointInterface</hardwareInterface>
     </joint>
     <actuator name="left_wheel2_motor">
