Commit message: change mass, in case the rover turns over

File: three_wheels_rover/robots_description/three_wheels_rover.gazebo.xacro (robot description, xacro)
@@ -13,5 +13,6 @@
       <legacyMode>true</legacyMode>
       <updateRate>100</updateRate>
-      <leftJoint>base_to_left</leftJoint> <!-- intentionally reverted -->
+      <rosDebugLevel>na</rosDebugLevel>
+      <leftJoint>base_to_left</leftJoint>
       <rightJoint>base_to_right</rightJoint>
       <wheelSeparation>0.474</wheelSeparation>
@@ -22,8 +23,14 @@
       <odometryTopic>odom</odometryTopic>
       <odometryFrame>odom</odometryFrame>
+      <odometrySource>world</odometrySource>
       <robotBaseFrame>base_footprint</robotBaseFrame>
-      <publishWheelTF>true</publishWheelTF>
+      <!--publishWheelTF>true</publishWheelTF--> <!--yuanye note: rviz will confuse with the parentlink-->
+      <publishTf>true</publishTf>
       <publishWheelJointState>true</publishWheelJointState>
     </plugin>
+  </gazebo>
+  <gazebo reference="base_footprint">
+    <mu1>0.1</mu1>
+    <mu2>0.1</mu2>
   </gazebo>
   <gazebo reference="base_link">
@@ -38,4 +45,6 @@
     <mu1>0.3</mu1>
     <mu2>0.3</mu2>
+    <kp>100000000.0</kp>
+    <kd>1.0</kd>
   </gazebo>
   <gazebo reference="tail_long">

File: three_wheels_rover/robots_description/three_wheels_rover.urdf.xacro (robot description, xacro)
@@ -196,5 +196,5 @@
     <type>transmission_interface/SimpleTransmission</type>
     <joint name="base_to_right">
-      <hardwareInterface>EffortJointInterface</hardwareInterface>
+      <hardwareInterface>hardware_interface/EffortJointInterface</hardwareInterface>
     </joint>
     <actuator name="right_wheel_motor">
@@ -204,8 +204,24 @@
     <type>transmission_interface/SimpleTransmission</type>
     <joint name="base_to_left">
-      <hardwareInterface>EffortJointInterface</hardwareInterface>
+      <hardwareInterface>hardware_interface/EffortJointInterface</hardwareInterface>
     </joint>
     <actuator name="left_wheel_motor">
     </actuator>
   </transmission>
+  <transmission name="tail_short_trans">
+    <type>transmission_interface/SimpleTransmission</type>
+    <joint name="tail_main_to_short">
+      <hardwareInterface>hardware_interface/EffortJointInterface</hardwareInterface>
+    </joint>
+    <actuator name="tail_short_motor">
+    </actuator>
+  </transmission>
+  <transmission name="rear_wheel_trans">
+    <type>transmission_interface/SimpleTransmission</type>
+    <joint name="tail_to_rear">
+      <hardwareInterface>hardware_interface/EffortJointInterface</hardwareInterface>
+    </joint>
+    <actuator name="rear_wheel_motor">
+    </actuator>
+  </transmission>
 </robot>
